File: hardware/canbus.sch (KiCad schematic (older format))
At the start: 21 parts, among them U201 MCP2551-I/SN, U202 MCP2515-xSO, Y201 16MHz

Commit message: layout
Parts:
- TP201, TP202, TP203, TP204, TP205, TP206, TP207, TP208, TP209: symbol Connector:TestPoint -> Connector:TestPoint_Probe
- U202: symbol MAB19-rescue:MCP2515-xSO-Interface_CAN_LIN -> Interface_CAN_LIN:MCP2515-xSO
Changed lines of the file:
@@
 EESchema Schematic File Version 4
-LIBS:MAB19-cache
-EELAYER 26 0
+EELAYER 30 0
 EELAYER END
 $Descr A4 11693 8268
@@
 EMI/ESD Protection Solutions for the CAN Bus: \nhttps://www.onsemi.com/pub/Collateral/AND8169-D.PDF\nSparkFun CAN-Bus Shield:\nhttps://cdn.sparkfun.com/datasheets/Dev/Arduino/Shields/SparkFun_CAN-Bus_Shield_v13a.pdf
 $Comp
-L Connector:TestPoint TP203
+L Connector:TestPoint_Probe TP203
 U 1 1 5AAC2327
 P 5550 3050
@@
 $EndComp
 $Comp
-L Connector:TestPoint TP204
+L Connector:TestPoint_Probe TP204
 U 1 1 5AAC23CC
 P 5550 3250
@@
 Connection ~ 5550 3200
 $Comp
-L Connector:TestPoint TP209
+L Connector:TestPoint_Probe TP209
 U 1 1 5AAC2B03
 P 5000 3650
@@
 $EndComp
 $Comp
-L Connector:TestPoint TP201
+L Connector:TestPoint_Probe TP201
 U 1 1 5AAC2C42
 P 3550 3000
@@
 $EndComp
 $Comp
-L Connector:TestPoint TP202
+L Connector:TestPoint_Probe TP202
 U 1 1 5AAC2C8C
 P 3400 3050
@@
 $EndComp
 $Comp
-L Connector:TestPoint TP206
+L Connector:TestPoint_Probe TP206
 U 1 1 5AAC2CDB
 P 3100 3550
@@
 $EndComp
 $Comp
-L Connector:TestPoint TP205
+L Connector:TestPoint_Probe TP205
 U 1 1 5AAC2E79
 P 3250 3450
@@
 Connection ~ 7650 3600
 $Comp
-L Connector:TestPoint TP208
+L Connector:TestPoint_Probe TP208
 U 1 1 5AAC8491
 P 8800 3600
@@
 $EndComp
 $Comp
-L Connector:TestPoint TP207
+L Connector:TestPoint_Probe TP207
 U 1 1 5AAC8C25
 P 7600 3600
@@
 Connection ~ 5550 4300
 $Comp
-L MAB19-rescue:MCP2515-xSO-Interface_CAN_LIN U202
+L Interface_CAN_LIN:MCP2515-xSO U202
 U 1 1 5BE69763
 P 4300 3700
-AR Path="/5BE69763" Ref="U202"  Part="1"
-AR Path="/5AABFC1B/5BE69763" Ref="U202"  Part="1"
 F 0 "U202" H 3850 4450 50  0000 C CNN
 F 1 "MCP2515-xSO" H 4650 2950 50  0000 C CNN
